Commit message: Cleaned up lewis description

File: rwi/b21_description/b21.xacro (robot description, xacro)
@@ -6,16 +6,8 @@
 	 name="lewis">
 <xacro:property name="thickness" value=".013" />
-<xacro:macro name="default_inertia" params="">
-	<inertial>
-		<mass value="1"/>
-		<inertia ixx="100" ixy="0" ixz="0" iyy="100" iyz="0" izz="100"/>
-		<origin/>
-	</inertial>
-</xacro:macro>
-<xacro:macro name="easy_cylinder" params="name radius length *vorigin *corigin *material">
+<xacro:macro name="easy_cylinder" params="name radius length *origin *material">
 <link name="${name}">
-	<xacro:default_inertia />
 	<visual>
-		<xacro:insert_block name="vorigin" />
+		<xacro:insert_block name="origin" />
 		<geometry>
 			<cylinder radius="${radius}" length="${length}" />
@@ -24,5 +16,5 @@
 	</visual>
 	<collision>
-		<xacro:insert_block name="corigin" />
+		<xacro:insert_block name="origin" />
 		<geometry>
 			<cylinder radius="${radius}" length="${length}" />
@@ -31,9 +23,8 @@
 </link>
 </xacro:macro>
-<xacro:macro name="easy_box" params="name size *vorigin *corigin *material">
+<xacro:macro name="easy_box" params="name size *origin *material">
 <link name="${name}">
-	<xacro:default_inertia />
 	<visual>
-		<xacro:insert_block name="vorigin" />
+		<xacro:insert_block name="origin" />
 		<geometry>
 			<box size="${size}" />
@@ -42,5 +33,5 @@
 	</visual>
 	<collision>
-		<xacro:insert_block name="corigin" />
+		<xacro:insert_block name="origin" />
 		<geometry>
 			<box size="${size}" />
@@ -58,5 +49,4 @@
 <xacro:easy_cylinder name="base" radius="0.26" length=".30">
 	<origin xyz="0 0 .15"/>
-	<origin xyz="0 0 .15"/>
 	<material name="lewisred">
 	<color rgba="1 0 0 1"/>
@@ -64,5 +54,4 @@
 </xacro:easy_cylinder>
 <xacro:easy_cylinder name="body" radius="0.25" length=".53">
-	<origin xyz="0 0 .265"/>
 	<origin xyz="0 0 .265"/>
 	<material name="lewisred" />
@@ -75,5 +64,5 @@
 </joint>
 <xacro:easy_box name="connector" size=".15 .30 .1">
-	<origin /><origin />
+	<origin />
 	<material name="black">
 		<color rgba="0 0 0 1"/>
@@ -84,5 +73,5 @@
 </xacro:fixedjoint>
 <xacro:easy_box name="laserbase" size=".04 .04 .04">
-	<origin /><origin />
+	<origin />
 	<material name="gray">
 		<color rgba=".8 .8 .8 1"/>
@@ -93,5 +82,5 @@
 </xacro:fixedjoint>
 <xacro:easy_cylinder name="laser" radius="0.02" length=".03">
-	<origin/><origin/>
+	<origin/>
 	<material name="black" />
 </xacro:easy_cylinder>
@@ -100,5 +89,5 @@
 </xacro:fixedjoint>
 <xacro:easy_cylinder name="bodytop" radius="0.25" length=".02">
-	<origin/><origin/>
+	<origin/>
 	<material name="black" />
 </xacro:easy_cylinder>
@@ -108,5 +97,5 @@
 <xacro:macro name="brace" params="prefix sign">
 	<xacro:easy_box name="${prefix}brace" size="0.1 .01 .13">
-		<origin /><origin />
+		<origin />
 		<material name="black" />
 	</xacro:easy_box>
@@ -118,5 +107,5 @@
 <xacro:brace prefix="right" sign="-" />
 <xacro:easy_box name="platform" size="0.30 .50 .06" >
-	<origin /><origin />
+	<origin />
 	<material name="lewisred"/>
 </xacro:easy_box>
@@ -125,5 +114,5 @@
 </xacro:fixedjoint>
 <xacro:easy_box name="graybase" size="0.14 .25 .005" >
-	<origin /><origin />
+	<origin />
 	<material name="gray"/>
 </xacro:easy_box>
@@ -133,5 +122,5 @@
 <xacro:macro name="post" params="num xsign ysign">
 	<xacro:easy_cylinder name="post${num}" length=".155" radius="0.005">
-		<origin /><origin />
+		<origin />
 		<material name="gray"/>
 	</xacro:easy_cylinder>
@@ -145,5 +134,5 @@
 <xacro:post num="4" xsign="-" ysign="-" />
 <xacro:easy_box name="graytop" size="0.135 .25 .005">
-	<origin/><origin/>
+	<origin/>
 	<material name="gray"/>
 </xacro:easy_box>
@@ -153,5 +142,4 @@
 <xacro:easy_box name="ptu_base" size="0.04 .07 .05">
 	<origin xyz="0 0.015 0"/>
-	<origin xyz="0 0.015 0"/>
 	<material name="black"/>
 </xacro:easy_box>
@@ -160,5 +148,5 @@
 </xacro:fixedjoint>
 <xacro:easy_box name="ptu_piece" size="0.04 .04 .06">
-	<origin/><origin/>
+	<origin/>
 	<material name="black"/>
 </xacro:easy_box>
@@ -170,5 +158,5 @@
 </joint>
 <xacro:easy_box name="ptu_mount" size="0.04 .27 .03">
-	<origin/><origin/>
+	<origin/>
 	<material name="gray"/>
 </xacro:easy_box>
@@ -181,5 +169,4 @@
 <xacro:macro name="eye" params="prefix sign">
 <link name="${prefix}eye">
-	<xacro:default_inertia />
 	<visual>
 		<geometry>

Commit message: Updated laser location

File: rwi/b21_description/b21.xacro (robot description, xacro)
@@ -79,5 +79,5 @@
 </xacro:easy_box>
 <xacro:fixedjoint name="tolaserbase" parent="body" child="laserbase">
-	<origin xyz="0.19 0 -.08"/>
+	<origin xyz="0 0 -.08"/>
 </xacro:fixedjoint>
 <xacro:easy_cylinder name="laser" radius="0.02" length=".03">

Commit message: Aligned laser

File: rwi/b21_description/b21.xacro (robot description, xacro)
@@ -79,5 +79,5 @@
 </xacro:easy_box>
 <xacro:fixedjoint name="tolaserbase" parent="body" child="laserbase">
-	<origin xyz="0 0 -.08"/>
+	<origin xyz="-0.29 0 -.08"/>
 </xacro:fixedjoint>
 <xacro:easy_cylinder name="laser" radius="0.02" length=".03">

Commit message: Change base_link of b21 description

File: rwi/b21_description/b21.xacro (robot description, xacro)
@@ -47,25 +47,32 @@
 </joint>
 </xacro:macro>
-<xacro:easy_cylinder name="base" radius="0.26" length=".30">
+<xacro:easy_cylinder name="base_link" radius="0.10" length=".30">
 	<origin xyz="0 0 .15"/>
-	<material name="lewisred">
-	<color rgba="1 0 0 1"/>
+	<material name="black">
+		<color rgba="0 0 0 1"/>
 	</material>
 </xacro:easy_cylinder>
 <xacro:easy_cylinder name="body" radius="0.25" length=".53">
 	<origin xyz="0 0 .265"/>
-	<material name="lewisred" />
+	<material name="lewisred">
+		<color rgba="1 0 0 1"/>
+	</material>
+</xacro:easy_cylinder>
+<xacro:fixedjoint name="base_to_body" parent="base_link" child="body">
+	<origin xyz="0 0 .40"/>
+</xacro:fixedjoint>
+<xacro:easy_cylinder name="base" radius="0.26" length=".30">
+	<origin xyz="0 0 .15"/>
+	<material name="lewisred"/>
 </xacro:easy_cylinder>
 <joint name="lewis_twist" type="continuous">
-	<parent link="base"/>
-	<child link="body"/>
-	<origin xyz="0 0 .40"/>
+	<parent link="body"/>
+	<child link="base"/>
+	<origin xyz="0 0 -.40"/>
 	<axis xyz="0 0 1"/>
 </joint>
 <xacro:easy_box name="connector" size=".15 .30 .1">
 	<origin />
-	<material name="black">
-		<color rgba="0 0 0 1"/>
-	</material>
+	<material name="black"/>
 </xacro:easy_box>
 <xacro:fixedjoint name="connect" parent="body" child="connector">
